File: plate/redherring-plate.kicad_pcb (KiCad board)
At the start: 2 copper layers, 364.4 x 144.6 mm, 86 parts

Commit message: Update with corrected placement and ISO Enter hotswap. Update plate - WIP
Parts:
- removed the REF** at (24.6, 328.6)
Other:
- outline, holes or cut-outs redrawn
